File: SensorKiCad-RTHMAT004/SensorKiCad-RTHMAT004.kicad_pcb (KiCad board)
At the start: 2 copper layers, 68 parts, among them J1 Conn_02x14_Odd_Even, J1 Conn_02x14_Odd_Even_MountingP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, Q1 SS8050, Q2 S5805, Q3 S5805, Q4 S5805, Q5 S5805, Q6 S5805

Commit message: Small changes to Sensor KiCAD file
Parts:
- removed the J1 at (200.0, -37.5)
- removed the J1 at (213.5, -33.5)
- added J1: Conn_02x14_Odd_Even, Connector_PinHeader_2.54mm:PinHeader_2x14_P2.54mm_Vertical, F.Cu at (50.9, 179.5)
- D2, D3, D4: footprint LED_THT:LED_D3.0mm_IRBlack -> LED_THT:LED_SideEmitter_Rectangular_W4.5mm_H1.6mm; moved to B.Cu
- Q2, Q3, Q4, Q5, Q6: value S5805 -> SS8050; footprint Package_TO_SOT_THT:TO-39-3 -> Package_TO_SOT_SMD:SOT-23
- R31, R32, R33: moved to B.Cu
- moved Q3 341.0 mm to (61.2, 136.2), turned to 90 degrees
- moved JP1 328.8 mm to (32.4, 164.0), turned to 180 degrees
- moved Q4 324.7 mm to (73.5, 136.4), turned to 90 degrees
- moved JP2 319.2 mm to (38.5, 164.0), turned to 180 degrees
- moved D1 317.3 mm to (31.3, 159.3), turned to 180 degrees
- moved Q2 316.8 mm to (41.1, 147.8), turned to 180 degrees
- moved JP3 313.3 mm to (43.4, 163.8), turned to 180 degrees
- moved Q5 311.8 mm to (91.2, 148.2)
- moved Q6 306.3 mm to (98.6, 159.0)
- moved JP4 302.3 mm to (40.6, 151.0)
- moved JP7 294.3 mm to (50.5, 134.7), turned to -90 degrees
- moved JP9 292.9 mm to (50.5, 139.8), turned to -90 degrees
- moved JP6 292.7 mm to (47.1, 151.0)
- moved JP8 290.9 mm to (64.3, 144.8), turned to -90 degrees
- moved JP5 288.4 mm to (47.0, 141.8)
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Connections:
- D6 pad 1: unconnected-(D6-K-Pad1) -> Net-(D6-K)
- JP11 pad 2: /PWM Left -> /PWM Centre
- JP14 pad 2: /PWM Left -> /PWM Right
- JP17 pad 2: /PWM Left -> /PWM Right
- JP2 pad 2: Net-(JP2-B) -> Net-(JP1-A)
- JP4 pad 1: unconnected-(JP4-A-Pad1) -> Net-(JP4-A)
- JP5 pad 1: unconnected-(JP5-A-Pad1) -> Net-(JP5-A)
- JP8 pad 2: /PWM Left -> /PWM Centre
- Q3 pad 1: unconnected-(Q3-E-Pad1) -> GND
- Q3 pad 3: unconnected-(Q3-C-Pad3) -> Net-(D6-K)
- R10 pad 1: unconnected-(R10-Pad1) -> Net-(JP5-A)
- R10 pad 2: unconnected-(R10-Pad2) -> Net-(Q2-B)
- R11 pad 1: /PWM Left -> /PWM Centre
- R16 pad 1: /PWM Left -> /PWM Centre
- R2 pad 1: Net-(JP2-B) -> Net-(JP1-A)
- R24 pad 1: /PWM Left -> /PWM Right
- R29 pad 1: /PWM Left -> /PWM Right
- R5 pad 2: unconnected-(R5-Pad2) -> Net-(Q1-B)
- R6 pad 1: unconnected-(R6-Pad1) -> Net-(JP4-A)
Routing:
- net /BATT: track 0.00 -> 247.9 mm
- net GND: track 0.00 -> 151.9 mm
- net /PWM Right: track 0.00 -> 87.3 mm
- net /Signal Left: track 0.00 -> 62.9 mm
- net /Signal Centre: track 0.00 -> 50.0 mm
- net /Signal Right: track 0.00 -> 38.1 mm
- net /PWM Centre: track 0.00 -> 36.2 mm
- net /PWM Left: track 0.00 -> 31.5 mm
- net Net-(D1-A): track 0.00 -> 25.7 mm
- net Net-(D9-A): track 0.00 -> 23.9 mm
- net Net-(D5-A): track 0.00 -> 23.6 mm
- net Net-(D8-A): track 0.00 -> 22.3 mm
- net Net-(D6-A): track 0.00 -> 20.5 mm
- net Net-(Q1-B): track 0.00 -> 16.6 mm
- net Net-(Q6-B): track 0.00 -> 14.9 mm
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
Commit message: Small changes to Sensor KiCAD file
Parts:
- D2, D3, D4, R31, R32, R33: moved to F.Cu
- moved D3 204.4 mm to (-21.1, -53.5), turned to 0 degrees
- moved D4 203.3 mm to (-55.3, -29.8)
- moved D8 203.3 mm to (11.2, -33.8)
- moved JP3 203.3 mm to (-44.0, -19.7)
- moved JP7 203.3 mm to (-36.8, -48.9)
- moved Q1 203.3 mm to (-51.5, -24.5)
- moved R16 203.3 mm to (-15.8, -37.6)
- moved R17 203.3 mm to (-15.9, -42.4)
- moved R4 203.3 mm to (-45.6, -23.7)
- moved R5 203.3 mm to (-42.2, -23.7)
- moved D1 203.3 mm to (-56.0, -24.3)
- moved D2 203.3 mm to (15.4, -28.8)
- moved D5 203.3 mm to (-51.6, -34.5)
- moved D6 203.3 mm to (-27.1, -51.8)
- moved D7 203.3 mm to (-15.1, -51.8)
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Routing:
- net /BATT: track 247.9 -> 106.2 mm
- net GND: track 151.9 -> 112.8 mm
- net /Signal Right: track 38.1 -> 74.0 mm
- net /Signal Centre: track 50.0 -> 23.9 mm
- net /Signal Left: track 62.9 -> 75.7 mm
- net /PWM Centre: track 36.2 -> 37.5 mm
- added copper zone on B.Cu, net GND

Commit message: Finalising PCB
Parts:
- added JP19: SolderJumper_2_Open, Jumper:SolderJumper-2_P1.3mm_Open_Pad1.0x1.5mm, F.Cu at (-1.00, -53.5)
- added JP20: SolderJumper_2_Open, Jumper:SolderJumper-2_P1.3mm_Open_Pad1.0x1.5mm, F.Cu at (-1.00, -48.8)
- added JP21: SolderJumper_2_Open, Jumper:SolderJumper-2_P1.3mm_Open_Pad1.0x1.5mm, F.Cu at (18.6, -16.6)
- added JP22: SolderJumper_2_Open, Jumper:SolderJumper-2_P1.3mm_Open_Pad1.0x1.5mm, F.Cu at (-1.00, -18.9)
- added JP23: SolderJumper_2_Open, Jumper:SolderJumper-2_P1.3mm_Open_Pad1.0x1.5mm, F.Cu at (-0.95, -16.1)
- added JP24: SolderJumper_2_Open, Jumper:SolderJumper-2_P1.3mm_Open_Pad1.0x1.5mm, F.Cu at (13.8, -16.5)
- added JP25: SolderJumper_2_Open, Jumper:SolderJumper-2_P1.3mm_Open_Pad1.0x1.5mm, F.Cu at (9.34, -16.6)
- added JP26: SolderJumper_2_Open, Jumper:SolderJumper-2_P1.3mm_Open_Pad1.0x1.5mm, F.Cu at (-2.10, -35.4)
- added JP27: SolderJumper_2_Open, Jumper:SolderJumper-2_P1.3mm_Open_Pad1.0x1.5mm, F.Cu at (7.65, -41.8)
- added JP28: SolderJumper_2_Open, Jumper:SolderJumper-2_P1.3mm_Open_Pad1.0x1.5mm, F.Cu at (7.65, -44.8)
- added JP29: SolderJumper_2_Open, Jumper:SolderJumper-2_P1.3mm_Open_Pad1.0x1.5mm, F.Cu at (-2.15, -29.9)
- added JP30: SolderJumper_2_Open, Jumper:SolderJumper-2_P1.3mm_Open_Pad1.0x1.5mm, F.Cu at (-2.21, -24.8)
- added JP31: SolderJumper_2_Open, Jumper:SolderJumper-2_P1.3mm_Open_Pad1.0x1.5mm, F.Cu at (-53.5, -31.0)
- added JP32: SolderJumper_2_Open, Jumper:SolderJumper-2_P1.3mm_Open_Pad1.0x1.5mm, F.Cu at (-43.5, -30.5)
- added JP33: SolderJumper_2_Open, Jumper:SolderJumper-2_P1.3mm_Open_Pad1.0x1.5mm, F.Cu at (-48.5, -31.0)
- added JP34: SolderJumper_2_Open, Jumper:SolderJumper-2_P1.3mm_Open_Pad1.0x1.5mm, F.Cu at (-21.8, -50.0)
- added JP35: SolderJumper_2_Open, Jumper:SolderJumper-2_P1.3mm_Open_Pad1.0x1.5mm, F.Cu at (-21.8, -40.0)
- added JP36: SolderJumper_2_Open, Jumper:SolderJumper-2_P1.3mm_Open_Pad1.0x1.5mm, F.Cu at (-21.8, -44.8)
- added JP37: SolderJumper_2_Open, Jumper:SolderJumper-2_P1.3mm_Open_Pad1.0x1.5mm, F.Cu at (3.50, -29.6)
- added JP38: SolderJumper_2_Open, Jumper:SolderJumper-2_P1.3mm_Open_Pad1.0x1.5mm, F.Cu at (8.30, -29.6)
- added JP39: SolderJumper_2_Open, Jumper:SolderJumper-2_P1.3mm_Open_Pad1.0x1.5mm, F.Cu at (13.7, -29.9)
- added R34: 100, Resistor_SMD:R_0805_2012Metric, F.Cu at (-46.0, -32.4)
- added R35: 1k, Resistor_SMD:R_1206_3216Metric, F.Cu at (-56.0, -33.0)
- added R36: 100, Resistor_SMD:R_0805_2012Metric, F.Cu at (-17.0, -39.0)
- added R37: 1k, Resistor_SMD:R_1206_3216Metric, F.Cu at (-17.5, -47.5)
- added R38: 100, Resistor_SMD:R_0805_2012Metric, F.Cu at (11.1, -32.4)
- added R39: 1k, Resistor_SMD:R_1206_3216Metric, F.Cu at (16.7, -31.9)
- added TP1: TestPoint, TestPoint:TestPoint_Pad_D2.5mm, F.Cu at (-36.5, -19.2)
- added TP2: TestPoint, TestPoint:TestPoint_Pad_D2.5mm, F.Cu at (-20.6, -36.3)
- added TP3: TestPoint, TestPoint:TestPoint_Pad_D2.5mm, F.Cu at (-6.20, -22.3)
- added TP4: TestPoint, TestPoint:TestPoint_Pad_D2.5mm, F.Cu at (-32.8, -17.0)
- added TP5: TestPoint, TestPoint:TestPoint_Pad_D2.5mm, F.Cu at (-32.7, -21.6)
- added TP6: TestPoint, TestPoint:TestPoint_Pad_D2.5mm, F.Cu at (-15.3, -23.0)
- added TP7: TestPoint, TestPoint:TestPoint_Pad_D2.5mm, F.Cu at (-6.40, -11.6)
- added TP8: TestPoint, TestPoint:TestPoint_Pad_D2.5mm, F.Cu at (-4.55, -15.9)
- D1, D5, D6, D7, D8, D9: footprint LED_THT:LED_D3.0mm_IRBlack -> LED_THT:LED_D5.0mm_Horizontal_O1.27mm_Z3.0mm_IRBlack
- JP1, JP10, JP11, JP12, JP13, JP14, JP15, JP16, JP17, JP18, JP2, JP3, JP4, JP5, JP6, JP7, JP8, JP9: value Jumper_2_Open -> SolderJumper_2_Open; footprint Jumper:SolderJumper-2_P1.3mm_Open_RoundedPad1.0x1.5mm -> Jumper:SolderJumper-2_P1.3mm_Open_Pad1.0x1.5mm
- R1, R15, R2, R20, R22, R27, R7: value 15 -> 47; footprint Resistor_SMD:R_0815_2038Metric -> Resistor_SMD:R_0805_2012Metric
- R10, R12, R17, R25: value 18k -> 47; footprint Resistor_SMD:R_0815_2038Metric -> Resistor_SMD:R_0805_2012Metric
- R11: value 8.2k -> 100; footprint Resistor_SMD:R_0815_2038Metric -> Resistor_SMD:R_0805_2012Metric
- R13, R18, R23, R28, R8: value 15 -> 8.2k; footprint Resistor_SMD:R_0815_2038Metric -> Resistor_SMD:R_0805_2012Metric
- R14, R19: value 15 -> 10k; footprint Resistor_SMD:R_0815_2038Metric -> Resistor_SMD:R_1206_3216Metric
- R16: value 8.2k. -> 100; footprint Resistor_SMD:R_0815_2038Metric -> Resistor_SMD:R_0805_2012Metric
- R21, R26, R3, R6: value 15 -> 100; footprint Resistor_SMD:R_0815_2038Metric -> Resistor_SMD:R_0805_2012Metric
- R24, R9: value 8.2k -> 10k; footprint Resistor_SMD:R_0815_2038Metric -> Resistor_SMD:R_1206_3216Metric
- R29: value 8.2 -> 10k; footprint Resistor_SMD:R_0815_2038Metric -> Resistor_SMD:R_1206_3216Metric
- R30: value 21 -> 47; footprint Resistor_SMD:R_0815_2038Metric -> Resistor_SMD:R_0805_2012Metric
- R31, R32, R33: value 21 -> 100; footprint Resistor_SMD:R_0815_2038Metric -> Resistor_SMD:R_0805_2012Metric
- R4: footprint Resistor_SMD:R_0815_2038Metric -> Resistor_SMD:R_0805_2012Metric
- R5: value 18k -> 10k; footprint Resistor_SMD:R_0815_2038Metric -> Resistor_SMD:R_1206_3216Metric
- moved JP15 45.9 mm to (-40.6, -51.8)
- moved JP14 38.6 mm to (-40.6, -43.2)
- moved JP13 35.1 mm to (-27.9, -29.2)
- moved JP10 35.0 mm to (-35.6, -25.0), turned to 0 degrees
- moved JP18 33.3 mm to (-17.2, -29.6), turned to 180 degrees
- moved R31 30.5 mm to (-51.0, -32.5), turned to -90 degrees
- moved R28 29.0 mm to (3.40, -41.8), turned to 180 degrees
- moved JP12 27.4 mm to (-28.0, -33.2), turned to 180 degrees
- moved JP16 26.0 mm to (-1.00, -43.8)
- moved R33 25.1 mm to (5.90, -32.4), turned to -90 degrees
- moved JP17 24.5 mm to (-17.2, -32.8), turned to 180 degrees
- moved JP11 22.9 mm to (-40.6, -47.5), turned to 180 degrees
- moved R24 22.4 mm to (3.50, -16.1), turned to 0 degrees
- moved JP5 21.1 mm to (-43.6, -21.0)
- moved R29 20.9 mm to (3.25, -44.8), turned to 180 degrees
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Connections:
- JP10 pad 2: Net-(JP10-B) -> /BATT
- JP11 pad 2: /PWM Centre -> /BATT
- JP12 pad 1: Net-(JP10-B) -> Net-(JP12-A)
- JP12 pad 2: /BATT -> /PWM Centre
- JP13 pad 2: Net-(JP13-B) -> /PWM Centre
- JP14 pad 2: /PWM Right -> /BATT
- JP15 pad 1: Net-(JP13-B) -> Net-(JP15-A)
- JP16 pad 2: Net-(JP16-B) -> /BATT
- JP17 pad 2: /PWM Right -> /PWM Centre
- JP18 pad 1: Net-(JP16-B) -> Net-(JP18-A)
- JP18 pad 2: /BATT -> /PWM Centre
- JP2 pad 2: Net-(JP1-A) -> /BATT
- JP3 pad 2: /PWM Left -> /BATT
- JP4 pad 2: Net-(JP4-B) -> /PWM Left
- JP6 pad 1: Net-(JP4-B) -> Net-(JP6-A)
- JP7 pad 2: Net-(JP7-B) -> /PWM Left
- JP8 pad 2: /PWM Centre -> /PWM Left
- JP9 pad 1: Net-(JP7-B) -> Net-(JP9-A)
- R1 pad 1: /BATT -> Net-(JP3-A)
- R10 pad 1: Net-(JP5-A) -> Net-(JP10-A)
- R10 pad 2: Net-(Q2-B) -> Net-(D5-A)
- R11 pad 1: /PWM Centre -> Net-(JP11-A)
- R11 pad 2: Net-(Q3-B) -> Net-(D6-A)
- R12 pad 1: Net-(JP8-A) -> Net-(JP14-A)
- R12 pad 2: Net-(Q3-B) -> Net-(D6-A)
- R13 pad 1: Net-(JP7-A) -> Net-(JP12-A)
- R13 pad 2: Net-(D6-A) -> Net-(Q3-B)
- R14 pad 1: Net-(JP7-B) -> Net-(JP13-A)
- R14 pad 2: Net-(D6-A) -> Net-(Q3-B)
- R15 pad 1: /BATT -> Net-(JP15-A)
- R16 pad 1: /PWM Centre -> Net-(JP16-A)
- R16 pad 2: Net-(Q4-B) -> Net-(D7-A)
- R17 pad 1: Net-(JP11-A) -> Net-(JP19-A)
- R17 pad 2: Net-(Q4-B) -> Net-(D7-A)
- R18 pad 1: Net-(JP10-A) -> Net-(JP17-A)
- R18 pad 2: Net-(D7-A) -> Net-(Q4-B)
- R19 pad 1: Net-(JP10-B) -> Net-(JP18-A)
- R19 pad 2: Net-(D7-A) -> Net-(Q4-B)
- R2 pad 1: Net-(JP1-A) -> Net-(JP2-A)
- R20 pad 1: /BATT -> Net-(JP20-A)
- R21 pad 1: Net-(JP13-A) -> Net-(JP21-A)
- R22 pad 1: Net-(JP13-B) -> Net-(JP24-A)
- R23 pad 1: /BATT -> Net-(JP22-A)
- R23 pad 2: Net-(D8-A) -> Net-(Q5-B)
- R24 pad 1: /PWM Right -> Net-(JP23-A)
- R25 pad 1: Net-(JP14-A) -> Net-(JP25-A)
- R25 pad 2: Net-(Q5-B) -> Net-(D8-A)
- R26 pad 1: Net-(JP16-A) -> Net-(JP26-A)
- R27 pad 1: Net-(JP16-B) -> Net-(JP29-A)
- R28 pad 1: /BATT -> Net-(JP27-A)
- R28 pad 2: Net-(D9-A) -> Net-(Q6-B)
- R29 pad 1: /PWM Right -> Net-(JP28-A)
- R3 pad 1: Net-(JP2-A) -> Net-(JP1-A)
- R30 pad 1: Net-(JP17-A) -> Net-(JP30-A)
- R30 pad 2: Net-(Q6-B) -> Net-(D9-A)
- R31 pad 2: GND -> Net-(JP33-B)
- R32 pad 2: GND -> Net-(JP36-B)
- R33 pad 2: GND -> Net-(JP37-B)
- R4 pad 1: /PWM Left -> Net-(JP4-A)
- R5 pad 1: Net-(JP3-A) -> Net-(JP5-A)
- R6 pad 1: Net-(JP4-A) -> Net-(JP6-A)
- R7 pad 1: Net-(JP4-B) -> Net-(JP9-A)
- R8 pad 1: /BATT -> Net-(JP7-A)
- R8 pad 2: Net-(D5-A) -> Net-(Q2-B)
- R9 pad 1: /PWM Left -> Net-(JP8-A)
Routing:
- net /BATT: track 106.2 -> 215.8 mm
- net GND: track 112.8 -> 47.5 mm
- net /PWM Left: track 31.5 -> 94.0 mm
- net /PWM Right: track 87.3 -> 46.6 mm
- net /Signal Centre: track 23.9 -> 50.9 mm
- net /PWM Centre: track 37.5 -> 47.7 mm
- net /Signal Left: track 75.7 -> 67.2 mm
- net Net-(JP10-B): track 8.13 -> 0.00 mm
- net Net-(JP7-B): track 7.83 -> 0.00 mm
- net Net-(D1-A): track 25.7 -> 17.9 mm
- net /Signal Right: track 74.0 -> 81.3 mm
- net Net-(JP13-B): track 7.08 -> 0.00 mm
- net Net-(JP4-B): track 6.96 -> 0.00 mm
- net Net-(JP16-B): track 6.83 -> 0.00 mm
- net Net-(D9-A): track 23.9 -> 30.6 mm
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- added copper zone on F.Cu, net GND

Commit message: pcb advancements
Parts:
- removed TP8: TestPoint, TestPoint:TestPoint_Pad_D2.5mm
- D1, D5, D6, D7, D8, D9: value SFH4544 -> SFH_4544; footprint LED_THT:LED_D5.0mm_Horizontal_O1.27mm_Z3.0mm_IRBlack -> SFH_4544:DIO_SFH_4544
- D2, D3, D4: footprint LED_THT:LED_SideEmitter_Rectangular_W4.5mm_H1.6mm -> BPV22NF:XDCR_BPV22NF
- moved TP5 25.0 mm to (-32.4, -46.6)
- moved JP34 4.15 mm to (-21.8, -45.9)
- moved TP7 3.32 mm to (-5.50, -14.8)
- moved D3 2.57 mm to (-19.1, -51.5), turned to 0 degrees
- moved R37 2.05 mm to (-17.6, -45.5)
- moved D5 2.00 mm to (-50.5, -38.3)
- moved JP36 1.95 mm to (-21.8, -42.8)
- moved D1 1.90 mm to (-50.6, -26.0)
- moved Q6 1.86 mm to (5.50, -37.7)
- moved Q2 1.85 mm to (-43.6, -39.0)
- moved R39 1.65 mm to (15.1, -31.9)
- moved TP3 1.64 mm to (-4.65, -21.8)
- moved D2 1.58 mm to (18.6, -31.0), turned to -90 degrees
- moved D6 1.53 mm to (-26.7, -43.7)
- moved D8 1.39 mm to (11.8, -24.7)
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Connections:
- J1 pad 10: /PWM Centre -> unconnected-(J1-Pin_10-Pad10)
- J1 pad 11: /Signal Right -> unconnected-(J1-Pin_11-Pad11)
- J1 pad 12: /PWM Right -> unconnected-(J1-Pin_12-Pad12)
- J1 pad 13: unconnected-(J1-Pin_13-Pad13) -> /Signal Centre
- J1 pad 15: unconnected-(J1-Pin_15-Pad15) -> GND
- J1 pad 16: unconnected-(J1-Pin_16-Pad16) -> /PWM Centre
- J1 pad 17: unconnected-(J1-Pin_17-Pad17) -> /Signal Right
- J1 pad 21: unconnected-(J1-Pin_21-Pad21) -> GND
- J1 pad 22: unconnected-(J1-Pin_22-Pad22) -> /PWM Right
- J1 pad 26: unconnected-(J1-Pin_26-Pad26) -> /BATT
- J1 pad 27: unconnected-(J1-Pin_27-Pad27) -> GND
- J1 pad 3: unconnected-(J1-Pin_3-Pad3) -> GND
- J1 pad 7: /Signal Centre -> unconnected-(J1-Pin_7-Pad7)
- Q1 pad 1: GND -> Net-(Q1-B)
- Q1 pad 2: Net-(Q1-B) -> GND
- Q1 pad 3: Net-(D1-K) -> Net-(Q1-C)
- Q2 pad 1: GND -> Net-(Q2-B)
- Q2 pad 2: Net-(Q2-B) -> GND
- Q2 pad 3: Net-(D5-K) -> Net-(Q2-C)
- Q3 pad 1: GND -> Net-(Q3-B)
- Q3 pad 2: Net-(Q3-B) -> GND
- Q3 pad 3: Net-(D6-K) -> Net-(Q3-C)
- Q4 pad 1: GND -> Net-(Q4-B)
- Q4 pad 2: Net-(Q4-B) -> GND
- Q4 pad 3: Net-(D7-K) -> Net-(Q4-C)
- Q5 pad 1: GND -> Net-(Q5-B)
- Q5 pad 2: Net-(Q5-B) -> GND
- Q5 pad 3: Net-(D8-K) -> Net-(Q5-C)
- Q6 pad 1: GND -> Net-(Q6-B)
- Q6 pad 2: Net-(Q6-B) -> GND
- Q6 pad 3: Net-(D9-K) -> Net-(Q6-C)
- R1 pad 2: Net-(D1-A) -> Net-(D1-PadA)
- R10 pad 2: Net-(D5-A) -> Net-(D5-PadA)
- R11 pad 2: Net-(D6-A) -> Net-(D6-PadA)
- R12 pad 2: Net-(D6-A) -> Net-(D6-PadA)
- R15 pad 2: Net-(D6-A) -> Net-(D6-PadA)
- R16 pad 2: Net-(D7-A) -> Net-(D7-PadA)
- R17 pad 2: Net-(D7-A) -> Net-(D7-PadA)
- R2 pad 2: Net-(D1-A) -> Net-(D1-PadA)
- R20 pad 2: Net-(D7-A) -> Net-(D7-PadA)
- R21 pad 2: Net-(D8-A) -> Net-(D8-PadA)
- R22 pad 2: Net-(D8-A) -> Net-(D8-PadA)
- R25 pad 2: Net-(D8-A) -> Net-(D8-PadA)
- R26 pad 2: Net-(D9-A) -> Net-(D9-PadA)
- R27 pad 2: Net-(D9-A) -> Net-(D9-PadA)
- R3 pad 2: Net-(D1-A) -> Net-(D1-PadA)
- R30 pad 2: Net-(D9-A) -> Net-(D9-PadA)
- R6 pad 2: Net-(D5-A) -> Net-(D5-PadA)
- R7 pad 2: Net-(D5-A) -> Net-(D5-PadA)
- TP5 pad 1: /PWM Left -> GND
Routing:
- net GND: track 47.5 -> 164.3 mm
- net /BATT: track 215.8 -> 287.4 mm
- net /PWM Right: track 46.6 -> 84.5 mm
- net Net-(D9-A): track 30.6 -> 0.00 mm
- net /PWM Centre: track 47.7 -> 75.3 mm
- net Net-(D9-PadA): track 0.00 -> 27.2 mm
- net Net-(D5-PadA): track 0.00 -> 23.6 mm
- net Net-(D5-A): track 23.0 -> 0.00 mm
- net Net-(D7-A): track 19.8 -> 0.00 mm
- net Net-(D8-A): track 19.1 -> 0.00 mm
- net /PWM Left: track 94.0 -> 75.4 mm
- net Net-(D1-A): track 17.9 -> 0.00 mm
- net Net-(D7-PadA): track 0.00 -> 17.5 mm
- net Net-(D1-PadA): track 0.00 -> 17.2 mm
- net Net-(D6-A): track 17.2 -> 0.00 mm
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Other:
- board outline added: 85 x 56 mm
- board text added: "Sensing Subsystem RTHMAT004, CLRMAT005"

Commit message: Final changes to sensor
Parts:
- added D10: BPV22NF, BPV22NF:XDCR_BPV22NF, F.Cu at (-15.4, -16.9)
- added Q7: SS8050, Package_TO_SOT_SMD:SOT-23, F.Cu at (-26.4, -22.4)
- added R40: 8.2k, Resistor_SMD:R_0805_2012Metric, F.Cu at (-22.0, -22.5)
- added R41: 10k, Resistor_SMD:R_1206_3216Metric, F.Cu at (-22.0, -18.1)
- added R42: 100, Resistor_SMD:R_0805_2012Metric, F.Cu at (-26.6, -18.0)
- added R43: 47, Resistor_SMD:R_0805_2012Metric, F.Cu at (-26.6, -14.2)
- added R44: 8.2k, Resistor_SMD:R_0805_2012Metric, F.Cu at (-10.8, -19.2)
- added R46: 100, Resistor_SMD:R_0805_2012Metric, F.Cu at (-10.9, -15.9)
- added R47: 47, Resistor_SMD:R_0805_2012Metric, F.Cu at (-10.9, -12.3)
- added R48: 8.2k, Resistor_SMD:R_0805_2012Metric, F.Cu at (-32.4, -17.3)
- added R50: 100, Resistor_SMD:R_0805_2012Metric, F.Cu at (-21.9, -13.2)
- added R51: 47, Resistor_SMD:R_0805_2012Metric, F.Cu at (-31.4, -13.9)
- added R52: 8.2k, Resistor_SMD:R_0805_2012Metric, F.Cu at (23.6, -20.4)
- added R53: 10k, Resistor_SMD:R_1206_3216Metric, F.Cu at (-10.7, -23.5)
- added R54: 100, Resistor_SMD:R_0805_2012Metric, F.Cu at (23.6, -16.9)
- added R55: 47, Resistor_SMD:R_0805_2012Metric, F.Cu at (23.6, -13.5)
- added TP10: TestPoint, TestPoint:TestPoint_Pad_D2.5mm, F.Cu at (-45.8, -14.8)
- added TP11: TestPoint, TestPoint:TestPoint_Pad_D2.5mm, F.Cu at (-62.8, -14.8)
- added TP8: TestPoint, TestPoint:TestPoint_Pad_D2.5mm, F.Cu at (-37.8, -14.0)
- D1, D5, D6, D7, D8, D9: footprint SFH_4544:DIO_SFH_4544 -> SFH_4544:LED_D5.0mm_Horizontal_O1.27mm_Z3.0mm_IRBlack_JLCPCB
- moved TP4 16.3 mm to (-31.8, -33.2)
- moved D9 5.33 mm to (6.50, -36.0)
- moved D5 4.85 mm to (-45.9, -39.6)
- moved Q6 2.60 mm to (2.90, -37.6)
- moved D7 1.30 mm to (-9.25, -43.9)
- moved D1 1.27 mm to (-50.6, -27.2)
- moved D4 1.25 mm to (-59.7, -32.1)
- moved JP4 1.25 mm to (-43.7, -18.2)
- moved R32 1.25 mm to (-15.8, -42.8)
- moved D6 1.20 mm to (-25.5, -43.8)
- moved D8 1.10 mm to (11.8, -23.6)
- moved R37 1.05 mm to (-16.5, -45.5)
- moved Q2 1.00 mm to (-42.6, -38.9)
- moved TP7 1.00 mm to (-4.50, -14.8)
- moved R25 0.86 mm to (8.00, -20.0)
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Routing:
- net GND: track 164.3 -> 23.2 mm, vias 0 -> 9
- net /PWM Centre: track 75.3 -> 48.3 mm, vias 0 -> 2
- net Net-(Q1-C): track 5.43 -> 22.2 mm
- net /PWM Right: track 84.5 -> 69.5 mm, vias 0 -> 2
- net Net-(D9-PadA): track 27.2 -> 22.4 mm
- net Net-(D5-PadA): track 23.6 -> 19.0 mm
- net Net-(Q1-B): track 11.1 -> 15.2 mm
- net /BATT: track 287.4 -> 283.4 mm
- net /PWM Left: track 75.4 -> 71.5 mm, vias 0 -> 2
- net Net-(Q2-C): track 6.16 -> 2.57 mm
- net Net-(D1-PadA): track 17.2 -> 20.5 mm
- net /Signal Centre: track 52.8 -> 56.0 mm
- net Net-(Q6-C): track 6.00 -> 3.55 mm
- net Net-(JP36-B): track 3.21 -> 4.46 mm
- net /Signal Right: track 94.5 -> 95.6 mm
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Other:
- board size 85 x 56 mm -> 95 x 57 mm

Commit message: Final changes to sensor
Parts:
- moved R55 3.79 mm to (19.8, -13.4)
- moved R52 1.48 mm to (22.1, -20.1)
- moved R54 0.25 mm to (23.3, -16.9)
Routing:
- net GND: track 23.2 -> 21.8 mm
- net /Signal Right: track 95.6 -> 94.7 mm
Other:
- board size 95 x 57 mm -> 93.5 x 57 mm

Commit message: Final changes to git repo
Parts:
- moved R10 206.4 mm to (133.3, 92.9)
- moved R6 206.4 mm to (133.3, 82.9)
- moved R7 206.4 mm to (133.3, 87.9)
- moved D1 206.4 mm to (120.6, 88.2)
- moved D10 206.4 mm to (155.8, 98.6)
- moved D2 206.4 mm to (190.4, 84.4)
- moved D3 206.4 mm to (152.1, 63.9)
- moved D4 206.4 mm to (111.5, 83.3)
- moved D5 206.4 mm to (125.3, 75.8)
- moved D6 206.4 mm to (145.7, 71.7)
- moved D7 206.4 mm to (161.9, 71.5)
- moved D8 206.4 mm to (183.0, 91.8)
- moved D9 206.4 mm to (177.7, 79.4)
- moved J1 206.4 mm to (134.8, 111.4)
- moved JP1 206.4 mm to (119.2, 94.4)
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Other:
- board text added: "PCB (other systems of micromouse)"
- board text added: "Servo- motor"
- board text added: "Wheel"
