File: SensorKiCad-RTHMAT004/SensorKiCad-RTHMAT004.kicad_sch (KiCad schematic)
At the start: 19 parts, among them J1 Conn_02x14_Odd_Even, Q1 SS8050

Commit message: Finalising PCB
Parts:
- added D5, D6, D7, D8, D9: SFH4544, LED_THT:LED_D5.0mm_Horizontal_O1.27mm_Z3.0mm_IRBlack, symbol LED:SFH4546
- added JP10, JP11, JP12, JP13, JP14, JP15, JP16, JP17, JP18, JP19, JP20, JP21, JP22, JP23, JP24, JP25, JP26, JP27, JP28, JP29, JP30, JP31, JP32, JP33, JP34, JP35, JP36, JP37, JP38, JP39, JP6, JP7, JP8, JP9: SolderJumper_2_Open, Jumper:SolderJumper-2_P1.3mm_Open_Pad1.0x1.5mm, symbol Jumper:SolderJumper_2_Open
- added Q2, Q3, Q4, Q5, Q6: SS8050, Package_TO_SOT_SMD:SOT-23, symbol Transistor_BJT:2N2219
- added R10, R12, R15, R17, R20, R22, R25, R27, R30, R7: 47, Resistor_SMD:R_0805_2012Metric, symbol Device:R_Small
- added R11, R16, R21, R26, R34, R36, R38, R6: 100, Resistor_SMD:R_0805_2012Metric, symbol Device:R_Small
- added R13, R18, R23, R28, R8: 8.2k, Resistor_SMD:R_0805_2012Metric, symbol Device:R_Small
- added R14, R19, R24, R29, R9: 10k, Resistor_SMD:R_1206_3216Metric, symbol Device:R_Small
- added R35, R37, R39: 1k, Resistor_SMD:R_1206_3216Metric, symbol Device:R_Small
- added TP1, TP2, TP3, TP4, TP5, TP6, TP7, TP8: TestPoint, TestPoint:TestPoint_Pad_D2.5mm, symbol Connector:TestPoint
- D1: footprint LED_THT:LED_D3.0mm_IRBlack -> LED_THT:LED_D5.0mm_Horizontal_O1.27mm_Z3.0mm_IRBlack
- D2, D3, D4: LCSC C2900370 -> C130226
- JP1, JP2, JP3, JP4, JP5: footprint (none) -> Jumper:SolderJumper-2_P1.3mm_Open_Pad1.0x1.5mm
- R1, R2: value 33 -> 47; footprint Resistor_SMD:R_0815_2038Metric -> Resistor_SMD:R_0805_2012Metric; LCSC (none) -> C17714
- R3: footprint Resistor_SMD:R_0815_2038Metric -> Resistor_SMD:R_0805_2012Metric; LCSC (none) -> C17901
- R31, R32, R33: value 21 -> 100; footprint Resistor_SMD:R_0815_2038Metric -> Resistor_SMD:R_0805_2012Metric; LCSC (none) -> C17901
- R4: footprint Resistor_SMD:R_0815_2038Metric -> Resistor_SMD:R_0805_2012Metric; LCSC (none) -> C17828
- R5: footprint Resistor_SMD:R_0815_2038Metric -> Resistor_SMD:R_1206_3216Metric; LCSC (none) -> C17902
Connections:
- net BATT: now also JP10.2 (B), JP11.2 (B), JP14.2 (B), JP15.2 (B), JP16.2 (B), JP19.2 (B), JP20.2 (B), JP21.2 (B), JP24.2 (B), JP25.2 (B), JP26.2 (B), JP29.2 (B), JP30.2 (B), JP6.2 (B), JP9.2 (B)
- net GND: now also JP31.1 (A), JP32.1 (A), JP33.1 (A), JP34.1 (A), JP35.1 (A), JP36.1 (A), JP37.1 (A), JP38.1 (A), JP39.1 (A), Q2.1 (E), Q3.1 (E), Q4.1 (E), Q5.1 (E), Q6.1 (E); no longer R31.2, R32.2, R33.2
- net PWM Centre: now also JP12.2 (B), JP13.2 (B), JP17.2 (B), JP18.2 (B), TP6.1
- net PWM Left: now also JP7.2 (B), JP8.2 (B), TP4.1, TP5.1
- net PWM Right: now also JP22.2 (B), JP23.2 (B), JP27.2 (B), JP28.2 (B), TP7.1, TP8.1
- net Signal Centre: now also R36.1, R37.1, TP2.1
- net Signal Left: now also R34.1, R35.1, TP1.1
- net Signal Right: now also R38.1, R39.1, TP3.1
- new net: JP35.2 (B), R36.2
- new net: Q3.2 (B), R13.2, R14.2
- new net: D6.1 (K), Q3.3 (C)
- new net: JP14.1 (A), R12.1
- new net: D6.2 (A), R11.2, R12.2, R15.2
- new net: JP9.1 (A), R7.1
- new net: D5.2 (A), R10.2, R6.2, R7.2
- new net: JP28.1 (A), R29.1
- new net: Q6.2 (B), R28.2, R29.2
- new net: JP12.1 (A), R13.1
- new net: JP32.2 (B), R34.2
- new net: JP26.1 (A), R26.1
- new net: JP37.2 (B), R33.2
- new net: JP31.2 (B), R35.2
- new net: JP23.1 (A), R24.1
- new net: Q5.2 (B), R23.2, R24.2
- new net: JP16.1 (A), R16.1
- new net: JP36.2 (B), R32.2
- new net: JP29.1 (A), R27.1
- new net: D9.2 (A), R26.2, R27.2, R30.2
- new net: JP38.2 (B), R38.2
- new net: JP27.1 (A), R28.1
- new net: JP39.2 (B), R39.2
- new net: JP6.1 (A), R6.1
- new net: JP21.1 (A), R21.1
- new net: JP25.1 (A), R25.1
- new net: JP7.1 (A), R8.1
- new net: JP19.1 (A), R17.1
- new net: D7.2 (A), R16.2, R17.2, R20.2
- new net: JP10.1 (A), R10.1
- new net: D9.1 (K), Q6.3 (C)
- new net: D7.1 (K), Q4.3 (C)
- new net: JP15.1 (A), R15.1
- new net: JP8.1 (A), R9.1
- new net: JP20.1 (A), R20.1
- new net: JP22.1 (A), R23.1
- new net: Q2.2 (B), R8.2, R9.2
- new net: D8.1 (K), Q5.3 (C)
- new net: JP24.1 (A), R22.1
- new net: JP33.2 (B), R31.2
- new net: JP18.1 (A), R19.1
- new net: JP34.2 (B), R37.2
- new net: JP11.1 (A), R11.1
- new net: D8.2 (A), R21.2, R22.2, R25.2
- new net: JP30.1 (A), R30.1
- new net: Q4.2 (B), R18.2, R19.2
- new net: D5.1 (K), Q2.3 (C)
- new net: JP17.1 (A), R18.1
- new net: JP13.1 (A), R14.1
Other:
- moved on the sheet: D2, D3, D4, JP1, JP2, JP3, JP4, JP5, Q1, R1, R2, R3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

Commit message: pcb advancements
Parts:
- removed D1, D5, D6, D7, D8, D9: SFH4544, LED_THT:LED_D5.0mm_Horizontal_O1.27mm_Z3.0mm_IRBlack, symbol LED:SFH4546
- removed D2, D3, D4: BPV22NF, LED_THT:LED_SideEmitter_Rectangular_W4.5mm_H1.6mm, symbol Device:D_Photo
- removed Q1, Q2, Q3, Q4, Q5, Q6: SS8050, Package_TO_SOT_SMD:SOT-23, symbol Transistor_BJT:2N2219
- removed TP8: TestPoint, TestPoint:TestPoint_Pad_D2.5mm, symbol Connector:TestPoint
- added D1, D5, D6, D7, D8, D9: SFH_4544, SFH_4544:DIO_SFH_4544, symbol SFH_4544:SFH_4544
- added D2, D3, D4: BPV22NF, BPV22NF:XDCR_BPV22NF, symbol BPV22NF:BPV22NF
- added Q1, Q2, Q3, Q4, Q5, Q6: SS8050, Package_TO_SOT_SMD:SOT-23, symbol Device:Q_NPN_BEC
Connections:
- net BATT: now also J1.26 (Pin_26), D2.K, D3.K, D4.K
- net GND: now also J1.15 (Pin_15), J1.21 (Pin_21), J1.27 (Pin_27), J1.3 (Pin_3), TP5.1, Q1.2 (E), Q2.2 (E), Q3.2 (E), Q4.2 (E), Q5.2 (E), Q6.2 (E)
- net PWM Centre: now also J1.16 (Pin_16); no longer J1.10 (Pin_10)
- net PWM Left: no longer TP5.1
- net PWM Right: now also J1.22 (Pin_22); no longer J1.12 (Pin_12)
- net Signal Centre: now also J1.13 (Pin_13), D3.A; no longer J1.7 (Pin_7)
- net Signal Left: now also D4.A
- net Signal Right: now also J1.17 (Pin_17), D2.A; no longer J1.11 (Pin_11)
- net at R13.2, R14.2: now also Q3.1 (B)
- net at R11.2, R12.2, R15.2: now also D6.A
- net at R10.2, R6.2, R7.2: now also D5.A
- net at R28.2, R29.2: now also Q6.1 (B)
- net at R4.2, R5.2: now also Q1.1 (B)
- net at R23.2, R24.2: now also Q5.1 (B)
- net at R26.2, R27.2, R30.2: now also D9.A
- net at R16.2, R17.2, R20.2: now also D7.A
- net at R1.2, R2.2, R3.2: now also D1.A
- net at R8.2, R9.2: now also Q2.1 (B)
- net at R21.2, R22.2, R25.2: now also D8.A
- net at R18.2, R19.2: now also Q4.1 (B)
- new net: D9.C, Q6.3 (C)
- new net: D7.C, Q4.3 (C)
- new net: D5.C, Q2.3 (C)
- new net: D1.C, Q1.3 (C)
- new net: D8.C, Q5.3 (C)
- new net: D6.C, Q3.3 (C)
Other:
- moved on the sheet: JP31, JP32, JP33, R31, R34, R35, TP1

Commit message: Final changes to sensor
Parts:
- added D10: BPV22NF, BPV22NF:XDCR_BPV22NF, symbol BPV22NF:BPV22NF
- added Q7: SS8050, Package_TO_SOT_SMD:SOT-23, symbol Device:Q_NPN_BEC
- added R40, R44, R48, R52: 8.2k, Resistor_SMD:R_0805_2012Metric, symbol Device:R_Small
- added R41, R53: 10k, Resistor_SMD:R_1206_3216Metric, symbol Device:R_Small
- added R42, R46, R50, R54: 100, Resistor_SMD:R_0805_2012Metric, symbol Device:R_Small
- added R43, R47, R51, R55: 47, Resistor_SMD:R_0805_2012Metric, symbol Device:R_Small
- added TP10, TP11, TP8: TestPoint, TestPoint:TestPoint_Pad_D2.5mm, symbol Connector:TestPoint
- D1, D5, D6, D7, D8, D9: footprint SFH_4544:DIO_SFH_4544 -> SFH_4544:LED_D5.0mm_Horizontal_O1.27mm_Z3.0mm_IRBlack_JLCPCB
Connections:
- net at Q1.1 (B), R4.2, R5.2: now also TP10.1
- net at D1.A, R1.2, R2.2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: now also TP11.1
- net at D1.C, Q1.3 (C): now also TP8.1
Other:
- moved on the sheet: D2, D3, D4, J1, JP31, JP32, JP33, JP34, JP35, JP36, JP37, JP38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

Commit message: Final changes to git repo
Connections:
- net 3V3: no longer names the net of J1.2 (Pin_2)
Other:
- note added: "- Emitter circuitry arranged from left to right. The left-most emitters on the schematic corellate to the emtters on the left side of the board. And the right most emitters on the schematic correlate to those on the right hand side of the board."
- note added: "- Emitter circuitry used for the emission of IR signals for the sensor circuitry as outlined in the report. - Sensor circuitry used for the sensing of the emitted signals subsequent to their reflection. It is the sensing of the reflected signal which will allow for sensing to occur."
- note added: "- Protection circuitry includes the following: - Jumpers (JPN) - Resistor arrangements (parallel banks enable resistance values to be changed for respective circuitry) - Multiple test points (TPN) for troubleshooting circuitry"
- note added: "- Signal Right, Signal Left, Signal Centre are each fed into the connector, corresponding to the ADC."
- note added: "- Similarly to the emitters, sensor circuitry has ben arranged from left to right as it would appear on the PCB."
- note added: "- The PWM Left, PWM Centre and PWM Right correspond to the pin on the connector for PWM allowing the emitters to be pulsed."
- note added: "Connector"
- note added: "Emitter Circuitry"
- note added: "Notes"
- note added: "Sensor Circuitry"
- note added: "Spare Components"
- company: (none) -> Matthew Rathbone
Changed lines of the file:
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@@
 	(title_block
 		(title "EEE3088F Sensing Board")
-		(date "2024-03-16")
-		(rev "v0")
+		(date "2024-04-10")
+		(rev "v3")
+		(company "Matthew Rathbone")
+		(comment 1 "EEE3088F - Sensor Subsystem")
+		(comment 2 "RTHMAT004")
 	)
 	(junction
@@
 		(pts
 			(xy 219.71 54.61) (xy 232.41 54.61)
-		)
-		(stroke
-			(width 0)
-			(type default)
-		)
-	)
-	(wire
-		(pts
-			(xy 256.54 36.83) (xy 245.11 36.83)
 		)
 		(stroke
@@
 	)
 	(rectangle
+		(start 13.97 156.21)
+		(end 175.26 195.58)
+		(stroke
+			(width 0)
+			(type default)
+		)
+		(fill
+			(type none)
+		)
+	)
+	(rectangle
 		(start 212.09 22.86)
 		(end 264.16 81.28)
@@
 		(fill
 			(type none)
+		)
+	)
+	(text "-	Protection circuitry includes the following:\n	- Jumpers (JPN)\n	- Resistor arrangements (parallel banks enable resistance values to be changed for respective circuitry)\n	- Multiple test points (TPN) for troubleshooting circuitry"
+		(exclude_from_sim no)
+		(at 14.732 173.99 0)
+		(effects
+			(font
+				(size 1.27 1.27)
+			)
+			(justify left)
+		)
+	)
+	(text "Spare Components"
+		(exclude_from_sim no)
+		(at 163.322 78.994 0)
+		(effects
+			(font
+				(size 1.905 1.905)
+			)
+		)
+	)
+	(text "Notes"
+		(exclude_from_sim no)
+		(at 18.542 158.75 0)
+		(effects
+			(font
+				(size 1.905 1.905)
+			)
+		)
+	)
+	(text "- 	Emitter circuitry arranged from left to right. The left-most emitters on the schematic corellate to the emtters on the left side of the board. And the right\n	most emitters on the schematic correlate to those on the right hand side of the board."
+		(exclude_from_sim no)
+		(at 14.732 163.576 0)
+		(effects
+			(font
+				(size 1.27 1.27)
+			)
+			(justify left)
+		)
+	)
+	(text "Emitter Circuitry"
+		(exclude_from_sim no)
+		(at 26.924 153.162 0)
+		(effects
+			(font
+				(size 1.905 1.905)
+			)
+		)
+	)
+	(text "-	Emitter circuitry used for the emission of IR signals for the sensor circuitry as outlined in the report. \n-	Sensor circuitry used for the sensing of the emitted signals subsequent to their reflection. It is the sensing of the reflected signal which will allow for \n	sensing to occur. \n"
+		(exclude_from_sim no)
+		(at 14.986 181.864 0)
+		(effects
+			(font
+				(size 1.27 1.27)
+			)
+			(justify left)
+		)
+	)
+	(text "Sensor Circuitry\n"
+		(exclude_from_sim no)
+		(at 40.386 79.502 0)
+		(effects
+			(font
+				(size 1.905 1.905)
+			)
+		)
+	)
+	(text "-	The PWM Left, PWM Centre and PWM Right correspond to the pin on the connector for PWM allowing the emitters to be pulsed. "
+		(exclude_from_sim no)
+		(at 14.986 188.976 0)
+		(effects
+			(font
+				(size 1.27 1.27)
+			)
+			(justify left)
+		)
+	)
+	(text "-	Similarly to the emitters, sensor circuitry has ben arranged from left to right as it would appear on the PCB."
+		(exclude_from_sim no)
+		(at 71.12 167.894 0)
+		(effects
+			(font
+				(size 1.27 1.27)
+			)
+		)
+	)
+	(text "Connector"
+		(exclude_from_sim no)
+		(at 220.218 79.756 0)
+		(effects
+			(font
+				(size 1.905 1.905)
+			)
+		)
+	)
+	(text "-	Signal Right, Signal Left, Signal Centre are each fed into the connector, corresponding to the ADC. "
+		(exclude_from_sim no)
+		(at 66.802 186.182 0)
+		(effects
+			(font
+				(size 1.27 1.27)
+			)
 		)
 	)
@@
 		)
 	)
-	(label "3V3"
-		(at 256.54 36.83 180)
-		(fields_autoplaced yes)
-		(effects
-			(font
-				(size 1.27 1.27)
-			)
-			(justify right bottom)
-		)
-	)
