File: PowerKiCad-CLRMAT005/PowerKiCad-CLRMAT005.kicad_sch (KiCad schematic)
At the start: 15 parts, among them J1 Conn_01x16_Pin, J2 Conn_01x02_Pin, SW1 SW_SPDT, U1 LEFT MOTOR, U2 RIGHT MOTOR, U3 MCP73831-2-OT

Commit message: added stuff to power subfolder
Other:
- note added: "16 pin connections of the power subsytem with their respective connections (not populated) ."
- note added: "2x1 pin connection for the battery (not populated)."
- note added: "MOTOR DRIVERS"
- note added: "Must be placed close to the pins on the PCB for heating reasons."
- note added: "OTHER"
- note added: "PIN CONNECTIONS"
- note added: "This circuit controls the two motors of the Micromouse."
- note added: "This circuit manages the charging of the battery from the 5V pin."
- note removed: "MOTOR DRIVER"
- note removed: "Must be placed close to the pins on the PCB"
- note removed: "PIN CONNECTIONS AND OTHER"
- note removed: "for heating reasons"
- title: Micro-mouse Power Subsytem -> Micromouse Power Subsytem
- moved on the sheet: R3, R4, SW1
Changed lines of the file:
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@@
 	(paper "A4")
 	(title_block
-		(title "Micro-mouse Power Subsytem")
+		(title "Micromouse Power Subsytem")
 		(date "2024-03-19")
-		(rev "v0")
+		(rev "v1.3")
 		(company "UCT EEE3088F")
 		(comment 1 "CLRMAT005")
@@
 	)
 	(junction
-		(at 99.06 64.77)
+		(at 179.07 64.77)
 		(diameter 0)
 		(color 0 0 0 0)
@@
 	(wire
 		(pts
-			(xy 107.95 36.83) (xy 115.57 36.83)
+			(xy 187.96 36.83) (xy 195.58 36.83)
 		)
 		(stroke
@@
 	(wire
 		(pts
-			(xy 99.06 71.12) (xy 99.06 73.66)
+			(xy 179.07 71.12) (xy 179.07 73.66)
 		)
 		(stroke
@@
 	(wire
 		(pts
-			(xy 115.57 36.83) (xy 115.57 39.37)
+			(xy 195.58 36.83) (xy 195.58 39.37)
 		)
 		(stroke
@@
 	(wire
 		(pts
-			(xy 107.95 31.75) (xy 115.57 31.75)
+			(xy 187.96 31.75) (xy 195.58 31.75)
 		)
 		(stroke
@@
 	(wire
 		(pts
-			(xy 99.06 64.77) (xy 99.06 66.04)
-		)
-		(stroke
-			(width 0)
-			(type default)
-		)
-	)
-	(wire
-		(pts
-			(xy 99.06 64.77) (xy 113.03 64.77)
+			(xy 179.07 64.77) (xy 179.07 66.04)
+		)
+		(stroke
+			(width 0)
+			(type default)
+		)
+	)
+	(wire
+		(pts
+			(xy 179.07 64.77) (xy 193.04 64.77)
 		)
 		(stroke
@@
 	(wire
 		(pts
-			(xy 87.63 34.29) (xy 97.79 34.29)
+			(xy 167.64 34.29) (xy 177.8 34.29)
 		)
 		(stroke
@@
 	(wire
 		(pts
-			(xy 99.06 53.34) (xy 99.06 57.15)
+			(xy 179.07 53.34) (xy 179.07 57.15)
 		)
 		(stroke
@@
 	(wire
 		(pts
-			(xy 99.06 62.23) (xy 99.06 64.77)
+			(xy 179.07 62.23) (xy 179.07 64.77)
 		)
 		(stroke
@@
 		)
 	)
-	(text "PIN CONNECTIONS AND OTHER\n"
+	(text "PIN CONNECTIONS\n"
 		(exclude_from_sim no)
 		(at 133.858 16.002 0)
 		(effects
 			(font
-				(size 1.27 1.27)
+				(size 2.032 2.032)
 				(bold yes)
 			)
 		)
 	)
+	(text "16 pin connections of the power subsytem with their \nrespective connections (not populated)\n."
+		(exclude_from_sim no)
+		(at 88.646 40.64 0)
+		(effects
+			(font
+				(size 1.27 1.27)
+			)
+		)
+	)
+	(text "2x1 pin connection for the battery (not populated).\n"
+		(exclude_from_sim no)
+		(at 87.122 73.66 0)
+		(effects
+			(font
+				(size 1.27 1.27)
+			)
+		)
+	)
 	(text "BATTERY CHARGER"
 		(exclude_from_sim no)
-		(at 273.05 93.218 0)
-		(effects
-			(font
-				(size 1.27 1.27)
+		(at 269.24 94.234 0)
+		(effects
+			(font
+				(size 2.032 2.032)
 				(bold yes)
 			)
 		)
 	)
-	(text "for heating reasons"
-		(exclude_from_sim no)
-		(at 162.306 97.79 0)
-		(effects
-			(font
-				(size 1.27 1.27)
-			)
-		)
-	)
-	(text "Must be placed close to the pins on the PCB"
-		(exclude_from_sim no)
-		(at 175.006 95.758 0)
-		(effects
-			(font
-				(size 1.27 1.27)
-			)
-		)
-	)
-	(text "MOTOR DRIVER"
-		(exclude_from_sim no)
-		(at 139.954 93.472 0)
-		(effects
-			(font
-				(size 1.27 1.27)
-				(thickness 0.254)
+	(text "This circuit manages the charging \nof the battery from the 5V pin.\n"
+		(exclude_from_sim no)
+		(at 172.466 137.16 0)
+		(effects
+			(font
+				(size 1.27 1.27)
+			)
+		)
+	)
+	(text "Must be placed close to the pins on the \nPCB for heating reasons."
+		(exclude_from_sim no)
+		(at 173.736 131.572 0)
+		(effects
+			(font
+				(size 1.27 1.27)
+			)
+		)
+	)
+	(text "This circuit controls the two motors \nof the Micromouse."
+		(exclude_from_sim no)
+		(at 129.286 114.808 0)
+		(effects
+			(font
+				(size 1.27 1.27)
+			)
+		)
+	)
+	(text "MOTOR DRIVERS"
+		(exclude_from_sim no)
+		(at 136.144 94.742 0)
+		(effects
+			(font
+				(size 1.778 1.778)
+				(bold yes)
+			)
+		)
+	)
+	(text "OTHER"
+		(exclude_from_sim no)
+		(at 277.368 16.764 0)
+		(effects
+			(font
+				(size 1.778 1.778)
+				(thickness 0.3556)
 				(bold yes)
 			)
@@
 	)
 	(label "BATT_ADC"
-		(at 113.03 64.77 0)
+		(at 193.04 64.77 0)
 		(fields_autoplaced yes)
 		(effects
@@
 	)
 	(label "BATT"
-		(at 99.06 53.34 0)
+		(at 179.07 53.34 0)
 		(fields_autoplaced yes)
 		(effects
@@
 	)
 	(label "BATT"
-		(at 115.57 31.75 0)
+		(at 195.58 31.75 0)
 		(fields_autoplaced yes)
 		(effects
@@
 	)
 	(label "BATT_IN"
-		(at 87.63 34.29 180)
+		(at 167.64 34.29 180)
 		(fields_autoplaced yes)
 		(effects
@@
 	(symbol
 		(lib_id "power:GND")
-		(at 99.06 73.66 0)
+		(at 179.07 73.66 0)
 		(unit 1)
 		(exclude_from_sim no)
@@
 		(fields_autoplaced yes)
 		(property "Reference" "#PWR014"
-			(at 99.06 80.01 0)
+			(at 179.07 80.01 0)
 			(effects
 				(font
@@
 		)
 		(property "Value" "GND"
-			(at 99.06 78.74 0)
+			(at 179.07 78.74 0)
 			(effects
 				(font
@@
 		)
 		(property "Footprint" ""
-			(at 99.06 73.66 0)
+			(at 179.07 73.66 0)
 			(effects
 				(font
@@
 		)
 		(property "Datasheet" ""
-			(at 99.06 73.66 0)
+			(at 179.07 73.66 0)
 			(effects
 				(font
@@
 		)
 		(property "Description" "Power symbol creates a global label with name \"GND\" , ground"
-			(at 99.06 73.66 0)
+			(at 179.07 73.66 0)
 			(effects
 				(font
@@
 	(symbol
 		(lib_id "power:GND")
-		(at 115.57 39.37 0)
+		(at 195.58 39.37 0)
 		(unit 1)
 		(exclude_from_sim no)
@@
 		(fields_autoplaced yes)
 		(property "Reference" "#PWR08"
-			(at 115.57 45.72 0)
+			(at 195.58 45.72 0)
 			(effects
 				(font
@@
 		)
 		(property "Value" "GND"
-			(at 115.57 44.45 0)
+			(at 195.58 44.45 0)
 			(effects
 				(font
@@
 		)
 		(property "Footprint" ""
-			(at 115.57 39.37 0)
+			(at 195.58 39.37 0)
 			(effects
 				(font
@@
 		)
 		(property "Datasheet" ""
-			(at 115.57 39.37 0)
+			(at 195.58 39.37 0)
 			(effects
 				(font
@@
 		)
 		(property "Description" "Power symbol creates a global label with name \"GND\" , ground"
-			(at 115.57 39.37 0)
+			(at 195.58 39.37 0)
 			(effects
 				(font
@@
 	(symbol
 		(lib_id "Switch:SW_SPDT")
-		(at 102.87 34.29 0)
+		(at 182.88 34.29 0)
 		(unit 1)
 		(exclude_from_sim no)
@@
 		(fields_autoplaced yes)
 		(property "Reference" "SW1"
-			(at 102.87 25.4 0)
+			(at 182.88 25.4 0)
 			(effects
 				(font
@@
 		)
 		(property "Value" "SW_SPDT"
-			(at 102.87 27.94 0)
+			(at 182.88 27.94 0)
 			(effects
 				(font
@@
 		)
 		(property "Footprint" "Button_Switch_THT:SW_Lever_1P2T_NKK_GW12LxH"
-			(at 102.87 34.29 0)
+			(at 182.88 34.29 0)
 			(effects
 				(font
@@
 		)
 		(property "Datasheet" "~"
-			(at 102.87 41.91 0)
+			(at 182.88 41.91 0)
 			(effects
 				(font
@@
 		)
 		(property "Description" "Switch, single pole double throw"
-			(at 102.87 34.29 0)
+			(at 182.88 34.29 0)
 			(effects
 				(font
@@
 	(symbol
 		(lib_id "Device:R_Small_US")
-		(at 99.06 59.69 0)
+		(at 179.07 59.69 0)
 		(unit 1)
 		(exclude_from_sim no)
@@
 		(fields_autoplaced yes)
 		(property "Reference" "R3"
-			(at 101.6 58.4199 0)
+			(at 181.61 58.4199 0)
 			(effects
 				(font
@@
 		)
 		(property "Value" "1.2k"
-			(at 101.6 60.9599 0)
+			(at 181.61 60.9599 0)
 			(effects
 				(font
@@
 		)
 		(property "Footprint" "Resistor_SMD:R_0805_2012Metric"
-			(at 99.06 59.69 0)
+			(at 179.07 59.69 0)
 			(effects
 				(font
@@
 		)
 		(property "Datasheet" "~"
-			(at 99.06 59.69 0)
+			(at 179.07 59.69 0)
 			(effects
 				(font
@@
 		)
 		(property "Description" "Resistor, small US symbol"
-			(at 99.06 59.69 0)
+			(at 179.07 59.69 0)
 			(effects
 				(font
@@
 	(symbol
 		(lib_id "Device:R_Small_US")
-		(at 99.06 68.58 0)
+		(at 179.07 68.58 0)
 		(unit 1)
 		(exclude_from_sim no)
@@
 		(fields_autoplaced yes)
 		(property "Reference" "R4"
-			(at 101.6 67.3099 0)
+			(at 181.61 67.3099 0)
 			(effects
 				(font
@@
 		)
 		(property "Value" "3k"
-			(at 101.6 69.8499 0)
+			(at 181.61 69.8499 0)
 			(effects
 				(font
@@
 		)
 		(property "Footprint" "Resistor_SMD:R_0603_1608Metric"
-			(at 99.06 68.58 0)
+			(at 179.07 68.58 0)
 			(effects
 				(font
@@
 		)
 		(property "Datasheet" "~"
-			(at 99.06 68.58 0)
+			(at 179.07 68.58 0)
 			(effects
 				(font
@@
 		)
 		(property "Description" "Resistor, small US symbol"
-			(at 99.06 68.58 0)
-			(effects
-				(font
+			(at 179.07 68.58 0)
+			(effects
+				(font
